File: pcb/mradio/5V_LDO.kicad_sch (KiCad schematic)
At the start: 15 parts, among them U205 TPS7A8500ARGRR

Commit message: Fixed passives
Parts:
- renumbered C231 to C501, C232 to C502, C233 to C503, C234 to C504, C235 to C505, C236 to C506, C237 to C507, C238 to C508, C239 to C509, C240 to C510, D204 to D501, R2 to R501, R1 to R502, R214 to R503, U205 to U501
Changed lines of the file:
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@@
 		(dnp no)
 		(fields_autoplaced yes)
-		(property "Reference" "#PWR0230"
+		(property "Reference" "#PWR0506"
 			(at 198.12 87.63 0)
 			(hide yes)
@@
 			(project "power_distribution"
 				(path "/e6698048-9125-4cf3-9b80-868e7e50deb6/4cca8186-706d-4229-b1ca-cabe637c5293"
-					(reference "#PWR0230")
+					(reference "#PWR0506")
 					(unit 1)
 				)
@@
 		(dnp no)
 		(fields_autoplaced yes)
-		(property "Reference" "R2"
+		(property "Reference" "R501"
 			(at 161.29 92.7099 0)
 			(show_name no)
@@
 			(project "power_distribution"
 				(path "/e6698048-9125-4cf3-9b80-868e7e50deb6/4cca8186-706d-4229-b1ca-cabe637c5293"
-					(reference "R2")
+					(reference "R501")
 					(unit 1)
 				)
@@
 		(dnp no)
 		(fields_autoplaced yes)
-		(property "Reference" "U205"
+		(property "Reference" "U501"
 			(at 138.43 50.8 0)
 			(show_name no)
@@
 			(project "power_distribution"
 				(path "/e6698048-9125-4cf3-9b80-868e7e50deb6/4cca8186-706d-4229-b1ca-cabe637c5293"
-					(reference "U205")
+					(reference "U501")
 					(unit 1)
 				)
@@
 		(dnp no)
 		(fields_autoplaced yes)
-		(property "Reference" "R1"
+		(property "Reference" "R502"
 			(at 176.53 83.8199 0)
 			(show_name no)
@@
 			(project "power_distribution"
 				(path "/e6698048-9125-4cf3-9b80-868e7e50deb6/4cca8186-706d-4229-b1ca-cabe637c5293"
-					(reference "R1")
+					(reference "R502")
 					(unit 1)
 				)
@@
 		(dnp no)
 		(fields_autoplaced yes)
-		(property "Reference" "C231"
+		(property "Reference" "C501"
 			(at 77.47 63.4999 0)
 			(show_name no)
@@
 			(project "power_distribution"
 				(path "/e6698048-9125-4cf3-9b80-868e7e50deb6/4cca8186-706d-4229-b1ca-cabe637c5293"
-					(reference "C231")
+					(reference "C501")
 					(unit 1)
 				)
@@
 		(dnp no)
 		(fields_autoplaced yes)
-		(property "Reference" "C236"
+		(property "Reference" "C506"
 			(at 162.56 83.8199 0)
 			(show_name no)
@@
 			(project "power_distribution"
 				(path "/e6698048-9125-4cf3-9b80-868e7e50deb6/4cca8186-706d-4229-b1ca-cabe637c5293"
-					(reference "C236")
+					(reference "C506")
 					(unit 1)
 				)
@@
 		(dnp no)
 		(fields_autoplaced yes)
-		(property "Reference" "C237"
+		(property "Reference" "C507"
 			(at 201.93 73.6599 0)
 			(show_name no)
@@
 			(project "power_distribution"
 				(path "/e6698048-9125-4cf3-9b80-868e7e50deb6/4cca8186-706d-4229-b1ca-cabe637c5293"
-					(reference "C237")
+					(reference "C507")
 					(unit 1)
 				)
@@
 		(dnp no)
 		(fields_autoplaced yes)
-		(property "Reference" "C240"
+		(property "Reference" "C510"
 			(at 237.49 73.6599 0)
 			(show_name no)
@@
 			(project "power_distribution"
 				(path "/e6698048-9125-4cf3-9b80-868e7e50deb6/4cca8186-706d-4229-b1ca-cabe637c5293"
-					(reference "C240")
+					(reference "C510")
 					(unit 1)
 				)
@@
 		(dnp no)
 		(fields_autoplaced yes)
-		(property "Reference" "C233"
+		(property "Reference" "C503"
 			(at 99.06 78.7399 0)
 			(show_name no)
@@
 			(project "power_distribution"
 				(path "/e6698048-9125-4cf3-9b80-868e7e50deb6/4cca8186-706d-4229-b1ca-cabe637c5293"
-					(reference "C233")
+					(reference "C503")
 					(unit 1)
 				)
@@
 		(dnp no)
 		(fields_autoplaced yes)
-		(property "Reference" "C235"
+		(property "Reference" "C505"
 			(at 105.41 86.3599 0)
 			(show_name no)
@@
 			(project "power_distribution"
 				(path "/e6698048-9125-4cf3-9b80-868e7e50deb6/4cca8186-706d-4229-b1ca-cabe637c5293"
-					(reference "C235")
+					(reference "C505")
 					(unit 1)
 				)
@@
 		(dnp no)
 		(fields_autoplaced yes)
-		(property "Reference" "#PWR0227"
+		(property "Reference" "#PWR0503"
 			(at 101.6 97.79 0)
 			(hide yes)
@@
 			(project "power_distribution"
 				(path "/e6698048-9125-4cf3-9b80-868e7e50deb6/4cca8186-706d-4229-b1ca-cabe637c5293"
-					(reference "#PWR0227")
+					(reference "#PWR0503")
 					(unit 1)
 				)
@@
 		(dnp no)
 		(fields_autoplaced yes)
-		(property "Reference" "D204"
+		(property "Reference" "D501"
 			(at 193.3575 55.88 0)
 			(show_name no)
@@
 			(project "power_distribution"
 				(path "/e6698048-9125-4cf3-9b80-868e7e50deb6/4cca8186-706d-4229-b1ca-cabe637c5293"
-					(reference "D204")
+					(reference "D501")
 					(unit 1)
 				)
@@
 		(dnp no)
 		(fields_autoplaced yes)
-		(property "Reference" "C234"
+		(property "Reference" "C504"
 			(at 100.33 63.4999 0)
 			(show_name no)
@@
 			(project "power_distribution"
 				(path "/e6698048-9125-4cf3-9b80-868e7e50deb6/4cca8186-706d-4229-b1ca-cabe637c5293"
-					(reference "C234")
+					(reference "C504")
 					(unit 1)
 				)
@@
 		(dnp no)
 		(fields_autoplaced yes)
-		(property "Reference" "#PWR0226"
+		(property "Reference" "#PWR0502"
 			(at 95.25 90.17 0)
 			(hide yes)
@@
 			(project "power_distribution"
 				(path "/e6698048-9125-4cf3-9b80-868e7e50deb6/4cca8186-706d-4229-b1ca-cabe637c5293"
-					(reference "#PWR0226")
+					(reference "#PWR0502")
 					(unit 1)
 				)
@@
 		(dnp no)
 		(fields_autoplaced yes)
-		(property "Reference" "C232"
+		(property "Reference" "C502"
 			(at 88.9 63.4999 0)
 			(show_name no)
@@
 			(project "power_distribution"
 				(path "/e6698048-9125-4cf3-9b80-868e7e50deb6/4cca8186-706d-4229-b1ca-cabe637c5293"
-					(reference "C232")
+					(reference "C502")
 					(unit 1)
 				)
@@
 		(dnp no)
 		(fields_autoplaced yes)
-		(property "Reference" "C239"
+		(property "Reference" "C509"
 			(at 226.06 73.6599 0)
 			(show_name no)
@@
 			(project "power_distribution"
 				(path "/e6698048-9125-4cf3-9b80-868e7e50deb6/4cca8186-706d-4229-b1ca-cabe637c5293"
-					(reference "C239")
+					(reference "C509")
 					(unit 1)
 				)
@@
 		(dnp no)
 		(fields_autoplaced yes)
-		(property "Reference" "#PWR0229"
+		(property "Reference" "#PWR0504"
 			(at 158.75 110.49 0)
 			(hide yes)
@@
 			(project "power_distribution"
 				(path "/e6698048-9125-4cf3-9b80-868e7e50deb6/4cca8186-706d-4229-b1ca-cabe637c5293"
-					(reference "#PWR0229")
+					(reference "#PWR0504")
 					(unit 1)
 				)
@@
 		(dnp no)
 		(fields_autoplaced yes)
-		(property "Reference" "#PWR0225"
+		(property "Reference" "#PWR0501"
 			(at 73.66 78.74 0)
 			(hide yes)
@@
 			(project "power_distribution"
 				(path "/e6698048-9125-4cf3-9b80-868e7e50deb6/4cca8186-706d-4229-b1ca-cabe637c5293"
-					(reference "#PWR0225")
+					(reference "#PWR0501")
 					(unit 1)
 				)
@@
 		(in_pos_files yes)
 		(dnp no)
-		(property "Reference" "#PWR0231"
+		(property "Reference" "#PWR0505"
 			(at 198.12 69.85 0)
 			(hide yes)
@@
 			(project "power_distribution"
 				(path "/e6698048-9125-4cf3-9b80-868e7e50deb6/4cca8186-706d-4229-b1ca-cabe637c5293"
-					(reference "#PWR0231")
+					(reference "#PWR0505")
 					(unit 1)
 				)
@@
 		(dnp no)
 		(fields_autoplaced yes)
-		(property "Reference" "R214"
+		(property "Reference" "R503"
 			(at 177.8 57.15 90)
 			(show_name no)
@@
 			(project "power_distribution"
 				(path "/e6698048-9125-4cf3-9b80-868e7e50deb6/4cca8186-706d-4229-b1ca-cabe637c5293"
-					(reference "R214")
+					(reference "R503")
 					(unit 1)
 				)
@@
 		(dnp no)
 		(fields_autoplaced yes)
-		(property "Reference" "C238"
+		(property "Reference" "C508"
 			(at 214.63 73.6599 0)
 			(show_name no)
@@
 			(project "power_distribution"
 				(path "/e6698048-9125-4cf3-9b80-868e7e50deb6/4cca8186-706d-4229-b1ca-cabe637c5293"
-					(reference "C238")
-					(unit 1)
-				)
+					(reference "C508")
+					(unit 1)
+				)
