File: pcb/mradio/ethernet.kicad_sch (KiCad schematic)
At the start: 22 parts, among them J301 RJ45_Wuerth_7499010211A, Q301 DN2540N3-G, U301 DP83825I, Y301 DSC1525JL2A-25M00000T

Commit message: some fixes, missing level shifter
Parts:
- removed C301: 0.01uF, symbol Device:C_Small
- removed Q301: DN2540N3-G, Package_TO_SOT_THT:TO-92_Inline, symbol Transistor_FET_Other:DN2540N3-G
- removed R301: 2.2k, Package_TO_SOT_THT:TO-92_Inline, symbol Device:R
- renumbered C306 to C1, C305 to C2, C304 to C3, C302 to C301, C310 to C302, C312 to C311, C303 to C4, C311 to C5, C309 to C6, C308 to C7, C307 to C8, FB301 to FB1, FB302 to FB2, J301 to J1, R303 to R1, R304 to R3, R305 to R5, U301 to U2
Connections:
- net ETH_RESET: now also U2.5 (~{RST})
- net GND: now also J1.11, J1.12
- no-connect marks 4 -> 2
Other:
- moved on the sheet: C301, R1, Y301

Commit message: ethernet edits
Parts:
- added C301: 0.01uF, symbol Device:C_Small
- added Q301: DN2540N3-G, Package_TO_SOT_THT:TO-92_Inline, symbol Transistor_FET_Other:DN2540N3-G
- added R301: 2.2k, Package_TO_SOT_THT:TO-92_Inline, symbol Device:R
- renumbered C301 to C302, C4 to C303, C3 to C304, C2 to C305, C1 to C306, C8 to C307, C7 to C308, C6 to C309, C302 to C310, C5 to C311, C311 to C312, FB1 to FB301, FB2 to FB302, J1 to J301, R1 to R303, R3 to R304, R5 to R305, U2 to U301
Connections:
- net ETH_RESET: now also Q301.2 (G); no longer U301.5 (~{RST})
- net GND: now also C301.2, R301.2; no longer J301.11, J301.12
- new net: Q301.1 (S), R301.1
- new net: C301.1, Q301.3 (D), U301.5 (~{RST})
- no-connect marks 2 -> 4
Other:
- moved on the sheet: C302, R303, Y301

Commit message: changed eth oscillator
Parts:
- removed C310, C312: 0.1uF, symbol Device:C_Small
- removed J301: RJ45_Wuerth_7499010211A, Connector_RJ:RJ45_Wuerth_7499010211A_Horizontal, symbol Connector:RJ45_Wuerth_7499010211A
- added C313, C314: 0.1uF, symbol Device:C_Small
- added J1: JX0026D21BNL, JX0026D21BNL:JX0026D21BNL, symbol symbols:JX0026D21BNL
- added R1: 70k, symbol Device:R_Small
- added TP1, TP2, TP3, TP301, TP302, TP303, TP4: TestPoint, symbol Connector:TestPoint
- R303: value (none) -> 2.2k
Connections:
- net +1V8: now also R1.1; no longer Y301.1 (OE)
- net ETH_RXD0: now also TP4.1
- net ETH_RXD1: now also TP3.1
- net ETH_TXD0: now also TP1.1
- net ETH_TXD1: now also TP2.1
- net GND: now also C313.1, C314.1, J1.12 (A_GREEN), J1.4 (CHS_GROUND_1), J1.5 (CHS_GROUND_2)
- net at C301.1, Q301.3 (D), U301.5 (~{RST}): now also TP303.1
- net at U301.11 (TD+): now also J1.1 (TD+)
- net at U301.10 (TD-): now also J1.2 (TD-)
- net at U301.8 (RD+): now also J1.7 (RD+)
- net at U301.7 (RD-): now also J1.8 (RD-)
- net at R305.1: now also J1.11 (K_GREEN)
- net at U301.13 (XI/50MHzIn), Y301.3 (OUT): now also TP302.1
- net at R304.1, U301.14 (RBIAS): now also TP301.1
- new net: R1.2, Y301.1 (OE)
- new net: C313.2, J1.3 (CT_1)
- new net: C314.2, J1.6 (CT_2)
- no-connect marks 4 -> 6
Other:
- moved on the sheet: R304
