File: pcb/mradio/5v5_Buck.kicad_sch (KiCad schematic)
At the start: 19 parts, among them U203 TPS54560BDDA

Commit message: Fixed passives
Parts:
- renumbered C202 to C401, C205 to C402, C210 to C403, C212 to C404, C214 to C405, C217 to C406, C223 to C407, C225 to C408, C227 to C409, C229 to C410, D202 to D401, L201 to L401, R201 to R401, R202 to R402, R205 to R403, R207 to R404, R210 to R405, R211 to R406, U203 to U401
Changed lines of the file:
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@@
 		(dnp no)
 		(fields_autoplaced yes)
-		(property "Reference" "R202"
+		(property "Reference" "R402"
 			(at 105.41 78.7399 0)
 			(show_name no)
@@
 			(project "power_distribution"
 				(path "/e6698048-9125-4cf3-9b80-868e7e50deb6/acb636b0-b919-4b86-a74c-b533f89957a8"
-					(reference "R202")
+					(reference "R402")
 					(unit 1)
 				)
@@
 		(dnp no)
 		(fields_autoplaced yes)
-		(property "Reference" "C202"
+		(property "Reference" "C401"
 			(at 53.34 65.4049 0)
 			(show_name no)
@@
 			(project "power_distribution"
 				(path "/e6698048-9125-4cf3-9b80-868e7e50deb6/acb636b0-b919-4b86-a74c-b533f89957a8"
-					(reference "C202")
+					(reference "C401")
 					(unit 1)
 				)
@@
 		(dnp no)
 		(fields_autoplaced yes)
-		(property "Reference" "R205"
+		(property "Reference" "R403"
 			(at 134.62 73.6599 0)
 			(show_name no)
@@
 			(project "power_distribution"
 				(path "/e6698048-9125-4cf3-9b80-868e7e50deb6/acb636b0-b919-4b86-a74c-b533f89957a8"
-					(reference "R205")
+					(reference "R403")
 					(unit 1)
 				)
@@
 		(dnp no)
 		(fields_autoplaced yes)
-		(property "Reference" "R211"
+		(property "Reference" "R406"
 			(at 257.81 95.2499 0)
 			(show_name no)
@@
 			(project "power_distribution"
 				(path "/e6698048-9125-4cf3-9b80-868e7e50deb6/acb636b0-b919-4b86-a74c-b533f89957a8"
-					(reference "R211")
+					(reference "R406")
 					(unit 1)
 				)
@@
 		(dnp no)
 		(fields_autoplaced yes)
-		(property "Reference" "C223"
+		(property "Reference" "C407"
 			(at 187.96 64.7699 0)
 			(show_name no)
@@
 			(project "power_distribution"
 				(path "/e6698048-9125-4cf3-9b80-868e7e50deb6/acb636b0-b919-4b86-a74c-b533f89957a8"
-					(reference "C223")
+					(reference "C407")
 					(unit 1)
 				)
@@
 		(dnp no)
 		(fields_autoplaced yes)
-		(property "Reference" "#PWR0221"
+		(property "Reference" "#PWR0407"
 			(at 196.85 83.82 0)
 			(hide yes)
@@
 			(project "power_distribution"
 				(path "/e6698048-9125-4cf3-9b80-868e7e50deb6/acb636b0-b919-4b86-a74c-b533f89957a8"
-					(reference "#PWR0221")
+					(reference "#PWR0407")
 					(unit 1)
 				)
@@
 		(dnp no)
 		(fields_autoplaced yes)
-		(property "Reference" "R201"
+		(property "Reference" "R401"
 			(at 105.41 68.5799 0)
 			(show_name no)
@@
 			(project "power_distribution"
 				(path "/e6698048-9125-4cf3-9b80-868e7e50deb6/acb636b0-b919-4b86-a74c-b533f89957a8"
-					(reference "R201")
+					(reference "R401")
 					(unit 1)
 				)
@@
 		(dnp no)
 		(fields_autoplaced yes)
-		(property "Reference" "#PWR0202"
+		(property "Reference" "#PWR0401"
 			(at 41.91 67.31 0)
 			(hide yes)
@@
 			(project "power_distribution"
 				(path "/e6698048-9125-4cf3-9b80-868e7e50deb6/acb636b0-b919-4b86-a74c-b533f89957a8"
-					(reference "#PWR0202")
+					(reference "#PWR0401")
 					(unit 1)
 				)
@@
 		(dnp no)
 		(fields_autoplaced yes)
-		(property "Reference" "R210"
+		(property "Reference" "R405"
 			(at 257.81 80.0099 0)
 			(show_name no)
@@
 			(project "power_distribution"
 				(path "/e6698048-9125-4cf3-9b80-868e7e50deb6/acb636b0-b919-4b86-a74c-b533f89957a8"
-					(reference "R210")
+					(reference "R405")
 					(unit 1)
 				)
@@
 		(dnp no)
 		(fields_autoplaced yes)
-		(property "Reference" "C227"
+		(property "Reference" "C409"
 			(at 231.14 72.3899 0)
 			(show_name no)
@@
 			(project "power_distribution"
 				(path "/e6698048-9125-4cf3-9b80-868e7e50deb6/acb636b0-b919-4b86-a74c-b533f89957a8"
-					(reference "C227")
+					(reference "C409")
 					(unit 1)
 				)
@@
 		(dnp no)
 		(fields_autoplaced yes)
-		(property "Reference" "#PWR0218"
+		(property "Reference" "#PWR0406"
 			(at 163.83 85.09 0)
 			(hide yes)
@@
 			(project "power_distribution"
 				(path "/e6698048-9125-4cf3-9b80-868e7e50deb6/acb636b0-b919-4b86-a74c-b533f89957a8"
-					(reference "#PWR0218")
+					(reference "#PWR0406")
 					(unit 1)
 				)
@@
 		(dnp no)
 		(fields_autoplaced yes)
-		(property "Reference" "#PWR0216"
+		(property "Reference" "#PWR0405"
 			(at 147.32 88.9 0)
 			(hide yes)
@@
 			(project "power_distribution"
 				(path "/e6698048-9125-4cf3-9b80-868e7e50deb6/acb636b0-b919-4b86-a74c-b533f89957a8"
-					(reference "#PWR0216")
+					(reference "#PWR0405")
 					(unit 1)
 				)
@@
 		(dnp no)
 		(fields_autoplaced yes)
-		(property "Reference" "#PWR0210"
+		(property "Reference" "#PWR0403"
 			(at 102.87 92.71 0)
 			(hide yes)
@@
 			(project "power_distribution"
 				(path "/e6698048-9125-4cf3-9b80-868e7e50deb6/acb636b0-b919-4b86-a74c-b533f89957a8"
-					(reference "#PWR0210")
+					(reference "#PWR0403")
 					(unit 1)
 				)
@@
 		(dnp no)
 		(fields_autoplaced yes)
-		(property "Reference" "R207"
+		(property "Reference" "R404"
 			(at 149.86 77.4699 0)
 			(show_name no)
@@
 			(project "power_distribution"
 				(path "/e6698048-9125-4cf3-9b80-868e7e50deb6/acb636b0-b919-4b86-a74c-b533f89957a8"
-					(reference "R207")
+					(reference "R404")
 					(unit 1)
 				)
@@
 		(dnp no)
 		(fields_autoplaced yes)
-		(property "Reference" "L201"
+		(property "Reference" "L401"
 			(at 208.28 64.77 90)
 			(show_name no)
@@
 			(project "power_distribution"
 				(path "/e6698048-9125-4cf3-9b80-868e7e50deb6/acb636b0-b919-4b86-a74c-b533f89957a8"
-					(reference "L201")
+					(reference "L401")
 					(unit 1)
 				)
@@
 		(in_pos_files yes)
 		(dnp no)
-		(property "Reference" "C214"
+		(property "Reference" "C405"
 			(at 125.73 77.4699 0)
 			(show_name no)
@@
 			(project "power_distribution"
 				(path "/e6698048-9125-4cf3-9b80-868e7e50deb6/acb636b0-b919-4b86-a74c-b533f89957a8"
-					(reference "C214")
+					(reference "C405")
 					(unit 1)
 				)
@@
 		(dnp no)
 		(fields_autoplaced yes)
-		(property "Reference" "C210"
+		(property "Reference" "C403"
 			(at 81.28 66.0399 0)
 			(show_name no)
@@
 			(project "power_distribution"
 				(path "/e6698048-9125-4cf3-9b80-868e7e50deb6/acb636b0-b919-4b86-a74c-b533f89957a8"
-					(reference "C210")
+					(reference "C403")
 					(unit 1)
 				)
@@
 		(dnp no)
 		(fields_autoplaced yes)
-		(property "Reference" "#PWR0213"
+		(property "Reference" "#PWR0404"
 			(at 132.08 92.71 0)
 			(hide yes)
@@
 			(project "power_distribution"
 				(path "/e6698048-9125-4cf3-9b80-868e7e50deb6/acb636b0-b919-4b86-a74c-b533f89957a8"
-					(reference "#PWR0213")
+					(reference "#PWR0404")
 					(unit 1)
 				)
@@
 		(dnp no)
 		(fields_autoplaced yes)
-		(property "Reference" "C229"
+		(property "Reference" "C410"
 			(at 242.57 72.3899 0)
 			(show_name no)
@@
 			(project "power_distribution"
 				(path "/e6698048-9125-4cf3-9b80-868e7e50deb6/acb636b0-b919-4b86-a74c-b533f89957a8"
-					(reference "C229")
+					(reference "C410")
 					(unit 1)
 				)
@@
 		(dnp no)
 		(fields_autoplaced yes)
-		(property "Reference" "C217"
+		(property "Reference" "C406"
 			(at 135.89 81.2799 0)
 			(show_name no)
@@
 			(project "power_distribution"
 				(path "/e6698048-9125-4cf3-9b80-868e7e50deb6/acb636b0-b919-4b86-a74c-b533f89957a8"
-					(reference "C217")
+					(reference "C406")
 					(unit 1)
 				)
@@
 		(dnp no)
 		(fields_autoplaced yes)
-		(property "Reference" "D202"
+		(property "Reference" "D401"
 			(at 199.39 72.0724 90)
 			(show_name no)
@@
 			(project "power_distribution"
 				(path "/e6698048-9125-4cf3-9b80-868e7e50deb6/acb636b0-b919-4b86-a74c-b533f89957a8"
-					(reference "D202")
+					(reference "D401")
 					(unit 1)
 				)
@@
 		(dnp no)
 		(fields_autoplaced yes)
-		(property "Reference" "C205"
+		(property "Reference" "C402"
 			(at 68.58 66.0399 0)
 			(show_name no)
@@
 			(project "power_distribution"
 				(path "/e6698048-9125-4cf3-9b80-868e7e50deb6/acb636b0-b919-4b86-a74c-b533f89957a8"
-					(reference "C205")
+					(reference "C402")
 					(unit 1)
 				)
@@
 		(dnp no)
 		(fields_autoplaced yes)
-		(property "Reference" "C212"
+		(property "Reference" "C404"
 			(at 93.98 66.0399 0)
 			(show_name no)
@@
 			(project "power_distribution"
 				(path "/e6698048-9125-4cf3-9b80-868e7e50deb6/acb636b0-b919-4b86-a74c-b533f89957a8"
-					(reference "C212")
+					(reference "C404")
 					(unit 1)
 				)
@@
 		(dnp no)
 		(fields_autoplaced yes)
-		(property "Reference" "U203"
+		(property "Reference" "U401"
 			(at 163.83 55.88 0)
 			(show_name no)
@@
 			(project "power_distribution"
 				(path "/e6698048-9125-4cf3-9b80-868e7e50deb6/acb636b0-b919-4b86-a74c-b533f89957a8"
-					(reference "U203")
+					(reference "U401")
 					(unit 1)
 				)
@@
 		(dnp no)
 		(fields_autoplaced yes)
-		(property "Reference" "#PWR0205"
+		(property "Reference" "#PWR0402"
 			(at 49.53 82.55 0)
 			(hide yes)
@@
 			(project "power_distribution"
 				(path "/e6698048-9125-4cf3-9b80-868e7e50deb6/acb636b0-b919-4b86-a74c-b533f89957a8"
-					(reference "#PWR0205")
+					(reference "#PWR0402")
 					(unit 1)
 				)
@@
 		(dnp no)
 		(fields_autoplaced yes)
-		(property "Reference" "C225"
+		(property "Reference" "C408"
 			(at 219.71 72.3899 0)
 			(show_name no)
@@
 			(project "power_distribution"
 				(path "/e6698048-9125-4cf3-9b80-868e7e50deb6/acb636b0-b919-4b86-a74c-b533f89957a8"
-					(reference "C225")
+					(reference "C408")
 					(unit 1)
 				)
@@
 		(dnp no)
 		(fields_autoplaced yes)
-		(property "Reference" "#PWR0223"
+		(property "Reference" "#PWR0408"
 			(at 255.27 106.68 0)
 			(hide yes)
@@
 			(project "power_distribution"
 				(path "/e6698048-9125-4cf3-9b80-868e7e50deb6/acb636b0-b919-4b86-a74c-b533f89957a8"
-					(reference "#PWR0223")
-					(unit 1)
-				)
+					(reference "#PWR0408")
+					(unit 1)
+				)

Commit message: Voltage conversion
Parts:
- added TP3: 2v2_TP, Module:RaspberryPi_Pico_SMD, symbol Connector:TestPoint
- C405: value 100pF -> 180pF
- R403: value 9.1k -> 3.74k
- R405: value 53.6k -> 17.4k
Connections:
- net at C407.2, D401.1 (K), L401.1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: now also TP3.1
- net 5.5V_Buck_out renamed 2.2V_Buck_Out
