File: pcb/mradio/900_mhz.kicad_sch (KiCad schematic)
At the start: 20 parts, among them J401 MM60-52B1-E1-R650, U401 74AVC4T774, U402 74AVC4T774

Commit message: add bypass caps to level shifters
Parts:
- added C411, C412: 0.1uF, Capacitor_SMD:C_0603_1608Metric, symbol Device:C
Connections:
- net +1V8: now also C412.2
- net +3V3: now also C411.2
- net GND: now also C411.1, C412.1
