File: pcb/mradio/900_mhz.kicad_sch (KiCad schematic)
At the start: 22 parts, among them J401 MM60-52B1-E1-R650, U401 74AVC4T774, U402 74AVC4T774

Commit message: fix level shifter symbol
Parts:
- U401, U402: symbol 74AVC4T774QPWRQ1:74AVC4T774QPWRQ1 -> symbols:74AVC4T774QPWRQ1
Changed lines of the file:
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@@
 	)
 	(symbol
-		(lib_id "74AVC4T774QPWRQ1:74AVC4T774QPWRQ1")
+		(lib_id "symbols:74AVC4T774QPWRQ1")
 		(at 177.8 139.7 0)
 		(unit 1)
@@
 		)
 		(property "Footprint" "Package_SO:TSSOP-16_4.4x5mm_P0.65mm"
-			(at 177.8 139.7 0)
+			(at 178.054 151.892 0)
 			(hide yes)
 			(show_name no)
@@
 	)
 	(symbol
-		(lib_id "74AVC4T774QPWRQ1:74AVC4T774QPWRQ1")
+		(lib_id "symbols:74AVC4T774QPWRQ1")
 		(at 233.68 139.7 0)
 		(unit 1)
@@
 		)
 		(property "Footprint" "Package_SO:TSSOP-16_4.4x5mm_P0.65mm"
-			(at 233.68 139.7 0)
-			(hide yes)
-			(show_name no)
+			(at 233.934 151.892 0)
+			(hide yes)
+			(show_name no)

Commit message: Update some footprints
Parts:
- TP401, TP402, TP403, TP404, TP405: footprint TestPoint:TestPoint_Pad_D1.0mm -> TestPoint:TestPoint_Loop_D2.60mm_Drill0.9mm_Beaded
Changed lines of the file:
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@@
 			)
 		)
-		(property "Footprint" "TestPoint:TestPoint_Pad_D1.0mm"
+		(property "Footprint" "TestPoint:TestPoint_Loop_D2.60mm_Drill0.9mm_Beaded"
 			(at 179.07 93.98 0)
 			(hide yes)
@@
 			)
 		)
-		(property "Footprint" "TestPoint:TestPoint_Pad_D1.0mm"
+		(property "Footprint" "TestPoint:TestPoint_Loop_D2.60mm_Drill0.9mm_Beaded"
 			(at 201.93 93.98 0)
 			(hide yes)
@@
 			)
 		)
-		(property "Footprint" "TestPoint:TestPoint_Pad_D1.0mm"
+		(property "Footprint" "TestPoint:TestPoint_Loop_D2.60mm_Drill0.9mm_Beaded"
 			(at 223.52 93.98 0)
 			(hide yes)
@@
 			)
 		)
-		(property "Footprint" "TestPoint:TestPoint_Pad_D1.0mm"
+		(property "Footprint" "TestPoint:TestPoint_Loop_D2.60mm_Drill0.9mm_Beaded"
 			(at 201.93 102.87 0)
 			(hide yes)
@@
 			)
 		)
-		(property "Footprint" "TestPoint:TestPoint_Pad_D1.0mm"
+		(property "Footprint" "TestPoint:TestPoint_Loop_D2.60mm_Drill0.9mm_Beaded"
 			(at 179.07 102.87 0)
 			(hide yes)

Commit message: Add mounting holes
Parts:
- added H401, H402: MountingHole_Pad, MountingHole:MountingHole_2.7mm_M2.5_Pad, symbol Mechanical:MountingHole_Pad
Connections:
- net GND: now also H401.1, H402.1

Commit message: make test points smaller
Parts:
- TP401, TP402, TP403, TP404, TP405: footprint TestPoint:TestPoint_Loop_D2.60mm_Drill0.9mm_Beaded -> TestPoint:TestPoint_Loop_D1.80mm_Drill1.0mm_Beaded
Changed lines of the file:
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@@
 			)
 		)
-		(property "Footprint" "TestPoint:TestPoint_Loop_D2.60mm_Drill0.9mm_Beaded"
+		(property "Footprint" "TestPoint:TestPoint_Loop_D1.80mm_Drill1.0mm_Beaded"
 			(at 179.07 93.98 0)
 			(hide yes)
@@
 			)
 		)
-		(property "Footprint" "TestPoint:TestPoint_Loop_D2.60mm_Drill0.9mm_Beaded"
+		(property "Footprint" "TestPoint:TestPoint_Loop_D1.80mm_Drill1.0mm_Beaded"
 			(at 201.93 93.98 0)
 			(hide yes)
@@
 			)
 		)
-		(property "Footprint" "TestPoint:TestPoint_Loop_D2.60mm_Drill0.9mm_Beaded"
+		(property "Footprint" "TestPoint:TestPoint_Loop_D1.80mm_Drill1.0mm_Beaded"
 			(at 223.52 93.98 0)
 			(hide yes)
@@
 			)
 		)
-		(property "Footprint" "TestPoint:TestPoint_Loop_D2.60mm_Drill0.9mm_Beaded"
+		(property "Footprint" "TestPoint:TestPoint_Loop_D1.80mm_Drill1.0mm_Beaded"
 			(at 201.93 102.87 0)
 			(hide yes)
@@
 			)
 		)
-		(property "Footprint" "TestPoint:TestPoint_Loop_D2.60mm_Drill0.9mm_Beaded"
+		(property "Footprint" "TestPoint:TestPoint_Loop_D1.80mm_Drill1.0mm_Beaded"
 			(at 179.07 102.87 0)
 			(hide yes)

Commit message: finished component placement
Parts:
- removed C411, C412: 0.1uF, Capacitor_SMD:C_0603_1608Metric, symbol Device:C
