File: pcb/mradio/3v7_Buck.kicad_sch (KiCad schematic)
At the start: 20 parts, among them U601 TPS54560BDDA

Commit message: Buck footprint updates
Parts:
- C601: footprint (none) -> Capacitor_THT:CP_Radial_D8.0mm_P3.50mm
- C602, C603, C604, C605, C606, C607, C608, C609, C610: footprint (none) -> Capacitor_SMD:C_0603_1608Metric
- D601: footprint (none) -> Diode_SMD:D_SMC
- L601: footprint (none) -> Inductor_SMD:L_Bourns_SRN6045TA
- R601, R602, R603, R604, R605, R606: footprint (none) -> Resistor_SMD:R_0603_1608Metric
Connections:
- net 3.7V_Buck_out renamed +3V7

Commit message: Update some footprints
Parts:
- TP601: footprint Module:RaspberryPi_Pico_SMD -> TestPoint:TestPoint_Loop_D2.60mm_Drill0.9mm_Beaded
Changed lines of the file:
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@@
 			)
 		)
-		(property "Footprint" "Module:RaspberryPi_Pico_SMD"
+		(property "Footprint" "TestPoint:TestPoint_Loop_D2.60mm_Drill0.9mm_Beaded"
 			(at 209.55 60.96 0)
 			(hide yes)

Commit message: make test points smaller
Parts:
- TP601: footprint TestPoint:TestPoint_Loop_D2.60mm_Drill0.9mm_Beaded -> TestPoint:TestPoint_Loop_D1.80mm_Drill1.0mm_Beaded
Changed lines of the file:
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@@
 			)
 		)
-		(property "Footprint" "TestPoint:TestPoint_Loop_D2.60mm_Drill0.9mm_Beaded"
+		(property "Footprint" "TestPoint:TestPoint_Loop_D1.80mm_Drill1.0mm_Beaded"
 			(at 209.55 60.96 0)
 			(hide yes)
