File: pcb/mradio/mradio.kicad_pcb (KiCad board)
At the start: 4 copper layers, 150 x 75 mm, 189 parts, among them J202 Conn_01x02, J301 JX0026D21BNL, J401 MM60-52B1-E1-R650, J501 MDT420E01001, U1 STM32H745ZITx, U301 DP83825I, U401 74AVC4T774, U402 74AVC4T774, U502 SN74LVC1T45DRL, U601 TPS54560BDDA, U701 TPS54560BDDA, U801 TPS7A8500ARGRR, U901 TPS7A8500ARGRR, Y301 DSC1525JL2A-25M00000T

Commit message: finished component placement
Parts:
- removed C411, C412: 0.1uF, Capacitor_SMD:C_0603_1608Metric
- removed D2, D3, D4, D5, D6, D7, D8: LED, LED_SMD:LED_0603_1608Metric
- removed R306: 1M, Resistor_SMD:R_0603_1608Metric
- removed the TP301 at (129.6, 132.4)
- removed TP303, TP304, TP305, TP306, TP307: TestPoint, TestPoint:TestPoint_Loop_D1.80mm_Drill1.0mm_Beaded
- added C106: 4.7uF, Capacitor_SMD:C_0603_1608Metric, F.Cu at (97.2, 81.8)
- added D101: LED, LED_SMD:LED_0603_1608Metric, F.Cu at (107.5, 103.0)
- added D102: LED, LED_SMD:LED_0603_1608Metric, F.Cu at (107.5, 104.5)
- added D103: LED, LED_SMD:LED_0603_1608Metric, F.Cu at (86.2, 74.5)
- added D104: LED, LED_SMD:LED_0603_1608Metric, F.Cu at (52.0, 75.8)
- added D105: LED, LED_SMD:LED_0603_1608Metric, F.Cu at (53.5, 75.8)
- added D106: LED, LED_SMD:LED_0603_1608Metric, F.Cu at (50.5, 75.8)
- added D107: LED, LED_SMD:LED_0603_1608Metric, F.Cu at (87.8, 74.5)
- added J101: Conn_02x07_Odd_Even, FTSH-107:SAMTEC_FTSH-107-01-X-DV-K, F.Cu at (110.0, 57.2)
- added Q101: Q_NMOS, SSM3K56FS:SSM_TOS_REAL, F.Cu at (61.5, 78.3)
- added Q102: Q_NMOS, SSM3K56FS:SSM_TOS_REAL, F.Cu at (106.0, 100.8)
- added Q103: Q_NMOS, SSM3K56FS:SSM_TOS_REAL, F.Cu at (106.0, 106.8)
- added Q104: Q_NMOS, SSM3K56FS:SSM_TOS_REAL, F.Cu at (83.9, 76.0)
- added Q105: Q_NMOS, SSM3K56FS:SSM_TOS_REAL, F.Cu at (69.8, 79.2)
- added Q106: Q_NMOS, SSM3K56FS:SSM_TOS_REAL, F.Cu at (64.2, 79.4)
- added Q107: Q_NMOS, SSM3K56FS:SSM_TOS_REAL, F.Cu at (67.0, 78.2)
- added Q108: Q_NMOS, SSM3K56FS:SSM_TOS_REAL, F.Cu at (90.1, 76.0)
- C313: value 1nF, 1KV -> 0nF
- moved R103 118.6 mm to (99.0, 60.8)
- moved R102 118.2 mm to (123.8, 66.8)
- moved C107 117.8 mm to (117.0, 61.2), turned to 90 degrees
- moved C120 116.9 mm to (114.5, 62.0), turned to 180 degrees
- moved C108 116.0 mm to (123.8, 73.2)
- moved C117 115.1 mm to (123.8, 65.2)
- moved R104 114.9 mm to (97.2, 66.8), turned to 180 degrees
- moved C109 114.4 mm to (123.8, 78.2)
- moved R101 112.7 mm to (123.8, 70.2)
- moved Q301 108.9 mm to (82.0, 59.2), turned to 90 degrees
- moved C407 108.4 mm to (125.0, 95.0)
- moved R112 107.8 mm to (87.8, 77.5), turned to -90 degrees
- moved R111 107.7 mm to (50.5, 79.0), turned to -90 degrees
- moved C406 107.6 mm to (125.0, 93.5)
- moved C110 106.3 mm to (119.0, 87.8), turned to -90 degrees
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- renumbered MOSFET301 to Q301, TP302 to TP301
Connections:
- C313 pad 1: GND -> unconnected-(C313-Pad1)
- C313 pad 2: Net-(J301-CHS_GROUND_1) -> GND
- J301 pad 4: Net-(J301-CHS_GROUND_1) -> GND
- J301 pad 5: Net-(J301-CHS_GROUND_1) -> GND
- J301 pad MH1: unconnected-(J301-PadMH1) -> unconnected-(C313-Pad1)
- J301 pad MH2: unconnected-(J301-PadMH2) -> unconnected-(C313-Pad1)
- R106 pad 2: /MCU/SoS_LED2 -> +3V3
- R107 pad 2: /MCU/SoS_LED3 -> +3V3
- R108 pad 2: /MCU/SoS_LED4 -> +3V3
- R109 pad 2: /MCU/M4_DBG1 -> +3V3
- R110 pad 2: /MCU/M4_DBG2 -> +3V3
- R111 pad 2: /MCU/M7_DBG1 -> +3V3
- R112 pad 2: /MCU/M7_DBG2 -> +3V3
Routing:
- net +1V8: track 0.00 -> 2.12 mm
Other:
- board size 150 x 75 mm -> 138.8 x 75 mm

Commit message: update stackup and wifi net class
Parts:
- removed R509, R510, R511: 0, Resistor_SMD:R_0603_1608Metric
- added R501: 0, Resistor_SMD:R_0603_1608Metric, F.Cu at (123.8, 83.2)
- added R502: 0, Resistor_SMD:R_0603_1608Metric, F.Cu at (122.5, 84.8)
- added R503: 0, Resistor_SMD:R_0603_1608Metric, F.Cu at (113.8, 87.8)
- R305: value R -> 55
- moved R508 11.7 mm to (123.8, 81.8), turned to 180 degrees
- moved R506 11.2 mm to (112.2, 87.8)
- moved R507 5.48 mm to (123.8, 80.2), turned to 180 degrees
Connections:
- J501 pad 11: Net-(J501-Pad11) -> /2.4-5 Ghz/SDIO_CMD
- J501 pad 13: Net-(J501-Pad13) -> /2.4-5 Ghz/SDIO_D0
- J501 pad 15: Net-(J501-Pad15) -> /2.4-5 Ghz/SDIO_D1
- J501 pad 17: Net-(J501-Pad17) -> /2.4-5 Ghz/SDIO_D2
- J501 pad 19: Net-(J501-Pad19) -> /2.4-5 Ghz/SDIO_D3
- J501 pad 9: Net-(J501-Pad9) -> /2.4-5 Ghz/SDIO_CK
- R506 pad 1: Net-(J501-Pad19) -> /2.4-5 Ghz/SDIO_D0
- R506 pad 2: SDMMC1_D3 -> SDMMC1_D0
- R507 pad 1: Net-(J501-Pad17) -> /2.4-5 Ghz/SDIO_CMD
- R507 pad 2: SDMMC1_D2 -> SDMMC1_CMD
- R508 pad 1: Net-(J501-Pad15) -> /2.4-5 Ghz/SDIO_CK
- R508 pad 2: SDMMC1_D1 -> SDMMC1_CK

Commit message: changed eth magjack
Parts:
- J301: value JX0026D21BNL -> 2250065-1; footprint JX0026D21BNL:JX0026D21BNL -> 2250065-1:BEL_2250065-1
- R305: value 55 -> 250
- moved C313 12.0 mm to (68.5, 64.2)
- moved J301 10.8 mm to (55.8, 64.5), turned to -90 degrees
- moved C312 6.12 mm to (68.5, 60.5)
- moved R305 5.36 mm to (68.5, 72.5)
- moved C311 4.95 mm to (68.5, 66.0)
Connections:
- C311 pad 2: Net-(J301-CT_1) -> Net-(J301-TCT)
- C312 pad 2: Net-(J301-CT_2) -> Net-(J301-RCT)
- C313 pad 1: unconnected-(C313-Pad1) -> Net-(J301-SHIELD)
- J301 pad 1: Net-(J301-TD+) -> /Ethernet/ETH_RD+
- J301 pad 10: unconnected-(J301-K_YELLOW-Pad10) -> GND
- J301 pad 11: Net-(J301-K_GREEN) -> unconnected-(J301-Pad11)
- J301 pad 12: GND -> unconnected-(J301-Pad12)
- J301 pad 2: Net-(J301-TD-) -> /Ethernet/ETH_RD-
- J301 pad 3: Net-(J301-CT_1) -> Net-(J301-RCT)
- J301 pad 4: GND -> Net-(J301-TCT)
- J301 pad 5: GND -> /Ethernet/ETH_TD+
- J301 pad 6: Net-(J301-CT_2) -> /Ethernet/ETH_TD-
- J301 pad 7: Net-(J301-RD+) -> (no net)
- J301 pad 8: Net-(J301-RD-) -> GND
- J301 pad 9: unconnected-(J301-A_YELLOW-Pad9) -> Net-(J301-Pad9)
- R305 pad 1: Net-(J301-K_GREEN) -> Net-(J301-Pad9)
- U301 pad 10: Net-(J301-TD-) -> /Ethernet/ETH_TD-
- U301 pad 11: Net-(J301-TD+) -> /Ethernet/ETH_TD+
- U301 pad 7: Net-(J301-RD-) -> /Ethernet/ETH_RD-
- U301 pad 8: Net-(J301-RD+) -> /Ethernet/ETH_RD+

Commit message: MCU decoupling caps
Parts:
- removed R103, R104: 0, Resistor_SMD:R_0603_1608Metric
- added C121: 100nF, Capacitor_SMD:C_0603_1608Metric, F.Cu at (110.2, 61.2)
- added C122: 100nF, Capacitor_SMD:C_0603_1608Metric, F.Cu at (113.2, 61.2)
- added C123: 100nF, Capacitor_SMD:C_0603_1608Metric, F.Cu at (123.8, 65.2)
- moved C117 35.9 mm to (98.0, 90.2)
- moved J101 14.0 mm to (124.0, 57.5)
- moved C120 1.25 mm to (115.5, 61.2), turned to 90 degrees
- moved C101 1.06 mm to (106.2, 61.2), turned to 90 degrees
Connections:
- C102 pad 1: /MCU/VDDA -> +1V8
- C103 pad 1: /MCU/VDDA -> +1V8
- C104 pad 1: /MCU/VREFP -> +1V8
- C105 pad 1: /MCU/VREFP -> +1V8
- U1 pad 35: /MCU/VREFP -> +1V8
- U1 pad 36: /MCU/VDDA -> +1V8
Routing:
- net +1V8: track 2.12 -> 4.04 mm
