File: pcb/mradio/mradio.kicad_pcb (KiCad board)
At the start: 4 copper layers, 138.8 x 75 mm, 191 parts, among them J101 Conn_02x07_Odd_Even, J202 Conn_01x02, J301 2250065-1, J401 MM60-52B1-E1-R650, J501 MDT420E01001, Q101 Q_NMOS, Q102 Q_NMOS, Q103 Q_NMOS, Q104 Q_NMOS, Q105 Q_NMOS, Q106 Q_NMOS, Q107 Q_NMOS, Q108 Q_NMOS, Q301 SSM3K56FS_LF, U1 STM32H745ZITx, U301 DP83825I, U401 74AVC4T774, U402 74AVC4T774, U502 SN74LVC1T45DRL, U601 TPS54560BDDA, U701 TPS54560BDDA, U801 TPS7A8500ARGRR, U901 TPS7A8500ARGRR, Y301 DSC1525JL2A-25M00000T

Commit message: 6 layers
Other:
- copper layers 4 -> 6
Changed lines of the file:
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@@
 	(generator_version "10.0")
 	(general
-		(thickness 1.5842)
+		(thickness 1.5584)
 		(legacy_teardrops no)
 	)
@@
 		(4 "In1.Cu" signal)
 		(6 "In2.Cu" signal)
+		(8 "In3.Cu" signal)
+		(10 "In4.Cu" signal)
 		(2 "B.Cu" signal)
 		(9 "F.Adhes" user "F.Adhesive")
@@
 			(layer "dielectric 2"
 				(type "core")
-				(thickness 1.265)
+				(thickness 0.55)
 				(material "FR4")
 				(epsilon_r 4.5)
@@
 			)
 			(layer "dielectric 3"
+				(type "prepreg")
+				(thickness 0.1088)
+				(material "FR4")
+				(epsilon_r 4.5)
+				(loss_tangent 0.02)
+			)
+			(layer "In3.Cu"
+				(type "copper")
+				(thickness 0.0152)
+			)
+			(layer "dielectric 4"
+				(type "core")
+				(thickness 0.55)
+				(material "FR4")
+				(epsilon_r 4.5)
+				(loss_tangent 0.02)
+			)
+			(layer "In4.Cu"
+				(type "copper")
+				(thickness 0.0152)
+			)
+			(layer "dielectric 5"
 				(type "prepreg")
 				(thickness 0.0994)
@@
 		(capping no)
 		(filling no)
+		(zone_defaults)
 		(pcbplotparams
 			(layerselection 0x00000000_00000000_55555555_5755f5ff)

Commit message: work on SDIO a bit
Parts:
- moved R512 25.2 mm to (113.8, 90.8)
- moved R516 16.8 mm to (126.0, 79.5), turned to -90 degrees
- moved R514 16.4 mm to (124.8, 85.5)
- moved D503 15.2 mm to (144.4, 89.0), turned to 0 degrees
- moved C511 14.6 mm to (146.2, 68.0)
- moved C512 14.5 mm to (146.2, 85.2)
- moved H501 14.5 mm to (169.5, 76.8)
- moved J501 14.5 mm to (141.2, 76.8)
- moved TP502 14.5 mm to (132.2, 75.2)
- moved D502 14.3 mm to (144.4, 90.5), turned to 0 degrees
- moved R505 11.1 mm to (147.4, 89.0), turned to 180 degrees
- moved C514 10.5 mm to (133.9, 69.8), turned to -90 degrees
- moved R504 9.74 mm to (147.4, 90.5), turned to 180 degrees
- moved U502 9.43 mm to (133.2, 72.2)
- moved XTAL501 7.53 mm to (139.1, 64.2)
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Connections:
- R512 pad 2: SDMMC1_D0 -> /2.4-5 Ghz/SDIO_D0
- R513 pad 2: SDMMC1_D1 -> /2.4-5 Ghz/SDIO_D1
- R514 pad 2: SDMMC1_D2 -> /2.4-5 Ghz/SDIO_D2
- R515 pad 2: SDMMC1_D3 -> /2.4-5 Ghz/SDIO_D3
- R516 pad 2: SDMMC1_CMD -> /2.4-5 Ghz/SDIO_CMD
Routing:
- net +3V3: track 0.00 -> 9.33 mm
- net /2.4-5 Ghz/SDIO_D1: track 0.00 -> 4.17 mm
- net /2.4-5 Ghz/SDIO_D3: track 0.00 -> 2.99 mm
- net /2.4-5 Ghz/SDIO_D0: track 0.00 -> 2.06 mm
- net SDMMC1_D3: track 0.00 -> 1.97 mm
- net SDMMC1_D1: track 0.00 -> 1.97 mm
- net SDMMC1_D0: track 0.00 -> 1.97 mm
- net SDMMC1_CMD: track 0.00 -> 1.97 mm
- net SDMMC1_CK: track 0.00 -> 1.97 mm
- net SDMMC1_D2: track 0.00 -> 1.71 mm
- net /2.4-5 Ghz/SDIO_D2: track 0.00 -> 1.46 mm
- net /2.4-5 Ghz/SDIO_CMD: track 0.00 -> 1.46 mm
- net Net-(D503-A): track 0.00 -> 1.39 mm
- net Net-(D502-A): track 0.00 -> 1.39 mm
- net +1V8: track 4.04 -> 5.28 mm

Commit message: route sdio
Parts:
- moved C511 2.62 mm to (144.6, 70.0)
- moved C512 2.62 mm to (144.5, 87.2)
- moved C513 2.62 mm to (130.8, 71.8)
- moved C514 2.62 mm to (132.2, 71.8)
- moved D502 2.62 mm to (142.7, 92.5)
- moved D503 2.62 mm to (142.7, 91.0)
- moved H501 2.62 mm to (167.8, 78.8)
- moved J501 2.62 mm to (139.6, 78.8)
- moved R504 2.62 mm to (145.7, 92.5)
- moved R505 2.62 mm to (145.7, 91.0)
- moved R513 2.62 mm to (130.1, 83.8)
- moved TP501 2.62 mm to (130.2, 67.8)
- moved TP502 2.62 mm to (130.5, 77.2)
- moved U502 2.62 mm to (131.5, 74.2)
- moved XTAL501 2.62 mm to (137.4, 66.2)
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Routing:
- net /2.4-5 Ghz/SDIO_CK: track 0.00 -> 22.6 mm, vias 0 -> 2
- net /2.4-5 Ghz/SDIO_CMD: track 1.46 -> 22.6 mm, vias 0 -> 2
- net /2.4-5 Ghz/SDIO_D2: track 1.46 -> 22.6 mm, vias 0 -> 2
- net /2.4-5 Ghz/SDIO_D0: track 2.06 -> 22.7 mm, vias 0 -> 2
- net /2.4-5 Ghz/SDIO_D3: track 2.99 -> 22.6 mm, vias 0 -> 2
- net /2.4-5 Ghz/SDIO_D1: track 4.17 -> 23.1 mm, vias 0 -> 2

Commit message: gnd + power planes
Routing:
- net Net-(XTAL501-CLK_Out): track 0.00 -> 11.6 mm
- net /2.4-5 Ghz/M2_WL_REG_ON: track 0.00 -> 9.83 mm, vias 0 -> 2
- added copper zone on In2.Cu, net +1V8
- added copper zone on In3.Cu, net +3V3
- added copper zone on In1.Cu, net GND
- added copper zone on In4.Cu, net GND
Changed lines of the file:
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@@
+	)
+	(segment
+		(start 138.25 73.1875)
+		(end 140.8125 75.75)
+		(width 0.2)
+		(layer "F.Cu")
+		(net "Net-(XTAL501-CLK_Out)")
+	)
+	(segment
+		(start 138.25 66.25)
+		(end 138.25 73.1875)
+		(width 0.2)
+		(layer "F.Cu")
+		(net "Net-(XTAL501-CLK_Out)")
+	)
+	(segment
+		(start 140.8125 75.75)
+		(end 141.8375 75.75)
+		(width 0.2)
+		(layer "F.Cu")
+		(net "Net-(XTAL501-CLK_Out)")
+	)
+	(segment
+		(start 141.8375 74.25)
+		(end 140.25 74.25)
+		(width 0.2)
+		(layer "F.Cu")
+		(net "/2.4-5 Ghz/M2_WL_REG_ON")
+	)
+	(segment
+		(start 133 74.75)
+		(end 132.2125 74.75)
+		(width 0.2)
+		(layer "F.Cu")
+		(net "/2.4-5 Ghz/M2_WL_REG_ON")
+	)
+	(via
+		(at 133 74.75)
+		(size 0.6)
+		(drill 0.3)
+		(layers "F.Cu" "B.Cu")
+		(net "/2.4-5 Ghz/M2_WL_REG_ON")
+	)
+	(via
+		(at 140.25 74.25)
+		(size 0.6)
+		(drill 0.3)
+		(layers "F.Cu" "B.Cu")
+		(net "/2.4-5 Ghz/M2_WL_REG_ON")
+	)
+	(segment
+		(start 133.5 74.25)
+		(end 133 74.75)
+		(width 0.2)
+		(layer "B.Cu")
+		(net "/2.4-5 Ghz/M2_WL_REG_ON")
+	)
+	(segment
+		(start 140.25 74.25)
+		(end 133.5 74.25)
+		(width 0.2)
+		(layer "B.Cu")
+		(net "/2.4-5 Ghz/M2_WL_REG_ON")
 	)
 	(segment
@@
 			)
 		)
+	)
+	(zone
+		(layers "In1.Cu" "In2.Cu" "In3.Cu" "In4.Cu")
+		(hatch edge 0.5)
+		(connect_pads
+			(clearance 0)
+		)
+		(min_thickness 0.25)
+		(keepout
+			(tracks allowed)
+			(vias allowed)
+			(pads allowed)
+			(copperpour not_allowed)
+			(footprints allowed)
+		)
+		(placement
+			(enabled no)
+			(sheetname "/2.4-5 Ghz/")
+		)
+		(fill
+			(thermal_gap 0.5)
+			(thermal_bridge_width 0.5)
+			(island_removal_mode 0)
+		)
+		(polygon
+			(pts
+				(xy 48.748792 55) (xy 66.248792 55) (xy 66.248792 74.25) (xy 48.748792 74.25)
+			)
+		)
+	)
+	(zone
+		(net "GND")
+		(layers "In1.Cu" "In4.Cu")
+		(name "Ground Planes")
+		(hatch edge 0.5)
+		(connect_pads
+			(clearance 0.5)
+		)
+		(min_thickness 0.25)
+		(fill yes
+			(thermal_gap 0.5)
+			(thermal_bridge_width 0.5)
+			(island_removal_mode 0)
+		)
+		(polygon
+			(pts
+				(xy 37 42.5) (xy 196.25 42.75) (xy 196 132.75) (xy 36.5 132.75)
+			)
+		)
+	)
+	(zone
+		(net "+1V8")
+		(layer "In2.Cu")
+		(hatch edge 0.5)
+		(priority 2)
+		(connect_pads
+			(clearance 0.5)
+		)
+		(min_thickness 0.25)
+		(fill yes
+			(thermal_gap 0.5)
+			(thermal_bridge_width 0.5)
+			(island_removal_mode 0)
+		)
+		(polygon
+			(pts
+				(xy 37 42.5) (xy 196.5 42.75) (xy 196.25 132.75) (xy 36.5 132.75)
+			)
+		)
+	)
+	(zone
+		(net "+3V3")
+		(layer "In3.Cu")
+		(hatch edge 0.5)
+		(priority 1)
+		(connect_pads
+			(clearance 0.5)
+		)
+		(min_thickness 0.25)
+		(fill yes
+			(thermal_gap 0.5)
+			(thermal_bridge_width 0.5)
+			(island_removal_mode 0)
+		)
+		(polygon
+			(pts
+				(xy 37 42.5) (xy 196.5 42.75) (xy 196.25 132.75) (xy 36.5 132.75)
+			)
+		)

Commit message: route wifi and mcu stuff
Parts:
- moved TP503 8.22 mm to (141.0, 65.5)
Routing:
- net GND: track 0.00 -> 66.8 mm, vias 0 -> 61
- net +1V8: track 5.28 -> 57.3 mm, vias 0 -> 23
- net /MCU/VCAP: track 0.00 -> 42.2 mm
- net /MCU/STLINK_RX: track 0.00 -> 36.2 mm, vias 0 -> 2
- net /MCU/STLINK_TX: track 0.00 -> 32.4 mm, vias 0 -> 2
- net WL_DEV_WAKE: track 0.00 -> 31.7 mm
- net /MCU/SWDIO: track 0.00 -> 29.2 mm, vias 0 -> 2
- net /MCU/SWCLK: track 0.00 -> 26.8 mm, vias 0 -> 2
- net /MCU/NRST: track 0.00 -> 21.7 mm
- net WL_HOST_WAKE: track 0.00 -> 19.8 mm, vias 0 -> 3
- net /MCU/SWO: track 0.00 -> 14.2 mm
- net WL_REG_ON: track 0.00 -> 10.6 mm
- net Net-(D502-K): track 0.00 -> 10.1 mm
- net /2.4-5 Ghz/M2_WL_REG_ON: track 9.83 -> 18.9 mm
- net +3V3: track 9.33 -> 15.4 mm, vias 0 -> 6
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
Commit message: LEDs
Parts:
- moved Q104 77.3 mm to (158.3, 54.7), turned to 180 degrees
- moved D103 75.6 mm to (159.8, 57.0), turned to 180 degrees
- moved D107 73.8 mm to (159.8, 58.5), turned to 180 degrees
- moved R108 73.4 mm to (156.8, 57.0), turned to 180 degrees
- moved R112 71.6 mm to (156.8, 58.5), turned to 180 degrees
- moved Q108 69.8 mm to (158.3, 60.8), turned to 0 degrees
- moved D101 59.2 mm to (144.8, 57.0)
- moved D102 59.2 mm to (144.8, 58.5)
- moved Q102 59.2 mm to (143.3, 54.8)
- moved Q103 59.2 mm to (143.3, 60.8)
- moved R106 59.2 mm to (141.8, 57.0)
- moved R107 59.2 mm to (141.8, 58.5)
- moved D104 1.50 mm to (53.5, 75.8)
- moved D105 1.50 mm to (52.0, 75.8)
- moved R109 1.50 mm to (53.5, 79.0)
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Routing:
- net /MCU/SoS_LED4: track 0.00 -> 59.4 mm, vias 0 -> 4
- net /MCU/M7_DBG1: track 0.00 -> 57.1 mm, vias 0 -> 2
- net /MCU/M7_DBG2: track 0.00 -> 52.5 mm, vias 0 -> 2
- net /MCU/SoS_LED2: track 0.00 -> 48.8 mm
- net /MCU/SoS_LED1: track 0.00 -> 45.9 mm, vias 0 -> 2
- net /MCU/SoS_LED3: track 0.00 -> 42.1 mm, vias 0 -> 2
- net /MCU/M4_DBG2: track 0.00 -> 41.1 mm, vias 0 -> 2
- net /MCU/M4_DBG1: track 0.00 -> 40.7 mm, vias 0 -> 2
- net Net-(D104-K): track 0.00 -> 19.5 mm, vias 0 -> 2
- net Net-(D106-K): track 0.00 -> 18.6 mm, vias 0 -> 2
- net Net-(D105-K): track 0.00 -> 14.4 mm
- net Net-(D1-K): track 0.00 -> 7.61 mm
- net GND: track 66.8 -> 73.7 mm, vias 61 -> 67
- net +3V3: track 15.4 -> 22.0 mm, vias 6 -> 14
- net Net-(D103-K): track 0.00 -> 2.97 mm
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
Commit message: make things a bit closer
Parts:
- moved C601 7.60 mm to (64.2, 116.8)
- moved U801 7.60 mm to (68.5, 91.2)
- moved C605 7.60 mm to (69.5, 104.4)
- moved C606 7.60 mm to (69.5, 102.9)
- moved C608 7.60 mm to (61.0, 93.5)
- moved C609 7.60 mm to (62.5, 93.5)
- moved C610 7.60 mm to (64.0, 93.5)
- moved C701 7.60 mm to (89.9, 119.8)
- moved C702 7.60 mm to (94.8, 119.8)
- moved C703 7.60 mm to (94.8, 118.2)
- moved C704 7.60 mm to (94.8, 116.8)
- moved C705 7.60 mm to (95.0, 107.5)
- moved C706 7.60 mm to (95.0, 106.0)
- moved C707 7.60 mm to (92.8, 113.2)
- moved C708 7.60 mm to (86.8, 96.5)
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Routing:
- net /MCU/SoS_LED4: track 59.4 -> 52.6 mm
- net /MCU/SoS_LED2: track 48.8 -> 41.9 mm
- net /MCU/SoS_LED3: track 42.1 -> 35.3 mm
- net /MCU/SoS_LED1: track 45.9 -> 39.1 mm
Other:
- board size 138.8 x 75 mm -> 132.2 x 75 mm

Commit message: start 900 mhz
Routing:
- net GND: track 73.7 -> 117.4 mm, vias 67 -> 99
- net +3V3: track 22.0 -> 41.7 mm, vias 14 -> 23
- net +1V8: track 57.3 -> 64.1 mm, vias 23 -> 26
