File: pcb/mradio/2v2_Buck.kicad_sch (KiCad schematic)
At the start: 20 parts, among them U401 TPS54560BDDA

Commit message: Buck footprint updates
Parts:
- C701: renamed from C401; footprint (none) -> Capacitor_THT:CP_Radial_D8.0mm_P3.50mm
- C702: renamed from C402; footprint (none) -> Capacitor_SMD:C_0603_1608Metric
- C703: renamed from C403; footprint (none) -> Capacitor_SMD:C_0603_1608Metric
- C704: renamed from C404; footprint (none) -> Capacitor_SMD:C_0603_1608Metric
- C705: renamed from C405; footprint (none) -> Capacitor_SMD:C_0603_1608Metric
- C706: renamed from C406; footprint (none) -> Capacitor_SMD:C_0603_1608Metric
- C707: renamed from C407; footprint (none) -> Capacitor_SMD:C_0603_1608Metric
- C708: renamed from C408; footprint (none) -> Capacitor_SMD:C_0603_1608Metric
- C709: renamed from C409; footprint (none) -> Capacitor_SMD:C_0603_1608Metric
- C710: renamed from C410; footprint (none) -> Capacitor_SMD:C_0603_1608Metric
- D701: renamed from D401; footprint (none) -> Diode_SMD:D_SMC
- L701: renamed from L401; footprint (none) -> Inductor_SMD:L_Bourns_SRN6045TA
- R701: renamed from R401; footprint (none) -> Resistor_SMD:R_0603_1608Metric
- R702: renamed from R402; footprint (none) -> Resistor_SMD:R_0603_1608Metric
- R703: renamed from R403; footprint (none) -> Resistor_SMD:R_0603_1608Metric
- R704: renamed from R404; footprint (none) -> Resistor_SMD:R_0603_1608Metric
- R705: renamed from R405; footprint (none) -> Resistor_SMD:R_0603_1608Metric
- R706: renamed from R406; footprint (none) -> Resistor_SMD:R_0603_1608Metric
- renumbered TP3 to TP701, U401 to U701
Connections:
- net 2.2V_Buck_Out renamed +2V2

Commit message: Update some footprints
Parts:
- TP701: footprint Module:RaspberryPi_Pico_SMD -> TestPoint:TestPoint_Loop_D2.60mm_Drill0.9mm_Beaded
Changed lines of the file:
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@@
 			)
 		)
-		(property "Footprint" "Module:RaspberryPi_Pico_SMD"
+		(property "Footprint" "TestPoint:TestPoint_Loop_D2.60mm_Drill0.9mm_Beaded"
 			(at 201.93 69.85 0)
 			(hide yes)

Commit message: make test points smaller
Parts:
- TP701: footprint TestPoint:TestPoint_Loop_D2.60mm_Drill0.9mm_Beaded -> TestPoint:TestPoint_Loop_D1.80mm_Drill1.0mm_Beaded
Changed lines of the file:
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@@
 			)
 		)
-		(property "Footprint" "TestPoint:TestPoint_Loop_D2.60mm_Drill0.9mm_Beaded"
+		(property "Footprint" "TestPoint:TestPoint_Loop_D1.80mm_Drill1.0mm_Beaded"
 			(at 201.93 69.85 0)
 			(hide yes)

Commit message: Changed 2v2 testpoint net to actually be 2v2...
Connections:
- net +2V2: now also TP701.1
- net at C707.2, D701.1 (K), L701.1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: no longer TP701.1
Changed lines of the file:
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@@
 	(paper "A4")
+	(junction
+		(at 219.71 69.85)
+		(diameter 0)
+		(color 0 0 0 0)
+	)
 	(junction
 		(at 132.08 71.12)
@@
 	(wire
 		(pts
-			(xy 215.9 69.85) (xy 227.33 69.85)
+			(xy 215.9 69.85) (xy 219.71 69.85)
 		)
 		(stroke
@@
 		(pts
 			(xy 64.77 71.12) (xy 77.47 71.12)
+		)
+		(stroke
+			(width 0)
+			(type default)
+		)
+	)
+	(wire
+		(pts
+			(xy 219.71 69.85) (xy 227.33 69.85)
 		)
 		(stroke
@@
 	)
 	(symbol
+		(lib_id "Connector:TestPoint")
+		(at 219.71 69.85 0)
+		(unit 1)
+		(body_style 1)
+		(exclude_from_sim no)
+		(in_bom yes)
+		(on_board yes)
+		(in_pos_files yes)
+		(dnp no)
+		(fields_autoplaced yes)
+		(property "Reference" "TP701"
+			(at 222.25 65.2779 0)
+			(show_name no)
+			(do_not_autoplace no)
+			(effects
+				(font
+					(size 1.27 1.27)
+				)
+				(justify left)
+			)
+		)
+		(property "Value" "2v2_TP"
+			(at 222.25 67.8179 0)
+			(show_name no)
+			(do_not_autoplace no)
+			(effects
+				(font
+					(size 1.27 1.27)
+				)
+				(justify left)
+			)
+		)
+		(property "Footprint" "TestPoint:TestPoint_Loop_D1.80mm_Drill1.0mm_Beaded"
+			(at 224.79 69.85 0)
+			(hide yes)
+			(show_name no)
+			(do_not_autoplace no)
+			(effects
+				(font
+					(size 1.27 1.27)
+				)
+			)
+		)
+		(property "Datasheet" ""
+			(at 224.79 69.85 0)
+			(hide yes)
+			(show_name no)
+			(do_not_autoplace no)
+			(effects
+				(font
+					(size 1.27 1.27)
+				)
+			)
+		)
+		(property "Description" "test point"
+			(at 219.71 69.85 0)
+			(hide yes)
+			(show_name no)
+			(do_not_autoplace no)
+			(effects
+				(font
+					(size 1.27 1.27)
+				)
+			)
+		)
+		(pin "1"
+		)
+		(instances
+			(project "mradio"
+				(path "/2cc0edad-946a-464e-a48b-49648a6334ed/acb636b0-b919-4b86-a74c-b533f89957a8"
+					(reference "TP701")
+					(unit 1)
+				)
+			)
+		)
+	)
+	(symbol
 		(lib_id "power:GND")
 		(at 163.83 78.74 0)
@@
 					(unit 1)
 				)
-			)
-		)
-	)
-	(symbol
-		(lib_id "Connector:TestPoint")
-		(at 196.85 69.85 0)
-		(unit 1)
-		(body_style 1)
-		(exclude_from_sim no)
-		(in_bom yes)
-		(on_board yes)
-		(in_pos_files yes)
-		(dnp no)
-		(fields_autoplaced yes)
-		(property "Reference" "TP701"
-			(at 199.39 65.2779 0)
-			(show_name no)
-			(do_not_autoplace no)
-			(effects
-				(font
-					(size 1.27 1.27)
-				)
-				(justify left)
-			)
-		)
-		(property "Value" "2v2_TP"
-			(at 199.39 67.8179 0)
-			(show_name no)
-			(do_not_autoplace no)
-			(effects
-				(font
-					(size 1.27 1.27)
-				)
-				(justify left)
-			)
-		)
-		(property "Footprint" "TestPoint:TestPoint_Loop_D1.80mm_Drill1.0mm_Beaded"
-			(at 201.93 69.85 0)
-			(hide yes)
-			(show_name no)
-			(do_not_autoplace no)
-			(effects
-				(font
-					(size 1.27 1.27)
-				)
-			)
-		)
-		(property "Datasheet" ""
-			(at 201.93 69.85 0)
-			(hide yes)
-			(show_name no)
-			(do_not_autoplace no)
-			(effects
-				(font
-					(size 1.27 1.27)
-				)
-			)
-		)
-		(property "Description" "test point"
-			(at 196.85 69.85 0)
-			(hide yes)
-			(show_name no)
-			(do_not_autoplace no)
-			(effects
-				(font
-					(size 1.27 1.27)
-				)
-			)
-		)
-		(pin "1"
-		)
-		(instances
-			(project "mradio"
-				(path "/2cc0edad-946a-464e-a48b-49648a6334ed/acb636b0-b919-4b86-a74c-b533f89957a8"
-					(reference "TP701")
-					(unit 1)
-				)
-			)
-			(project "power_distribution"
-				(path "/e6698048-9125-4cf3-9b80-868e7e50deb6/acb636b0-b919-4b86-a74c-b533f89957a8"
-					(reference "TP3")
-					(unit 1)
-				)
