File: pcb/mradio/1v8_LDO.kicad_sch (KiCad schematic)
At the start: 16 parts, among them U501 TPS7A8500ARGRR

Commit message: Voltage conversion
Parts:
- removed C501: 47uF, RGR0020A, symbol Device:C
- removed C502, C503, C504: 10uF, RGR0020A, symbol Device:C
- removed C505: 100nF, symbol Device:C
- removed C506: 10nF, symbol Device:C
- removed C507: 47uF, symbol Device:C
- removed C508: 10uF, symbol Device:C
- removed C509: 1uF, symbol Device:C
- removed C510: 0.1uF, symbol Device:C
- removed D501: LED, symbol Device:LED
- removed R501: 2.37k, symbol Device:R
- removed R502: 12.4k, symbol Device:R
- removed R503: 1.2k, symbol Device:R
- removed TP2: 5V_TP, Module:RaspberryPi_Pico_SMD, symbol Connector:TestPoint
- removed U501: TPS7A8500ARGRR, RGR0020A, symbol symbols:TPS7A8500ARGRR
- added C511: 47uF, RGR0020A, symbol Device:C
- added C512, C513, C514: 10uF, RGR0020A, symbol Device:C
- added C515: 100nF, symbol Device:C
- added C516: 10nF, symbol Device:C
- added C517: 47uF, symbol Device:C
- added C518, C519, C520: 10uF, symbol Device:C
- added D502: LED, symbol Device:LED
- added R506: 1.2k, symbol Device:R
- added TP1: 1v8_TP, Module:RaspberryPi_Pico_SMD, symbol Connector:TestPoint
- added U502: TPS7A8500ARGRR, RGR0020A, symbol symbols:TPS7A8500ARGRR
Connections:
- net GND: now also C511.2, C512.2, C513.2, C514.2, C515.2, C517.2, C518.2, C519.2, C520.2, D502.1 (K), U502.10 (800_mV), U502.18 (GND), U502.21 (PAD), U502.7 (200_mV), U502.8 (GND)
- new net: C515.1, U502.13 (NR_SS)
- new net: C516.2, U502.3 (FB)
- new net: D502.2 (A), R506.1, U502.4 (PG)
- new net 1V8_LDO_Out: C516.1, C517.1, C518.1, C519.1, C520.1, TP1.1, U502.1 (OUT), U502.19 (OUT), U502.2 (SNS), U502.20 (OUT)
- new net 2V_Buck_or_3v3_LDO_Out: C511.1, C512.1, C513.1, C514.1, R506.2, U502.12 (BIAS), U502.14 (EN), U502.15 (IN), U502.16 (IN), U502.17 (IN)
- no-connect marks 6 -> 4

Commit message: Fixed passive numbers
Parts:
- renumbered C511 to C1001, C512 to C1002, C513 to C1003, C514 to C1004, C515 to C1005, C516 to C1006, C517 to C1007, C518 to C1008, C519 to C1009, C520 to C1010, D502 to D1001, R506 to R1001, TP1 to TP1001, U502 to U1001

Commit message: undid overwrite
Connections:
- net 2V_Buck_or_3v3_LDO_Out: no longer R1001.2
- new net 3v3_LDO_Out: R1001.2
Changed lines of the file:
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@@
+	)
+	(junction
+		(at 113.03 53.34)
+		(diameter 0)
+		(color 0 0 0 0)
 	)
 	(junction
@@
 	(wire
 		(pts
-			(xy 111.76 73.66) (xy 111.76 53.34)
-		)
-		(stroke
-			(width 0)
-			(type default)
-		)
-	)
-	(wire
-		(pts
 			(xy 67.31 81.28) (xy 67.31 85.09)
 		)
@@
 	(wire
 		(pts
-			(xy 111.76 53.34) (xy 128.27 53.34)
+			(xy 111.76 53.34) (xy 113.03 53.34)
 		)
 		(stroke
@@
 		(pts
 			(xy 215.9 83.82) (xy 226.06 83.82)
+		)
+		(stroke
+			(width 0)
+			(type default)
+		)
+	)
+	(wire
+		(pts
+			(xy 113.03 53.34) (xy 128.27 53.34)
 		)
 		(stroke
@@
 	(label "2V_Buck_or_3v3_LDO_Out"
 		(at 67.31 73.66 180)
+		(effects
+			(font
+				(size 1.27 1.27)
+			)
+			(justify right bottom)
+		)
+	)
+	(label "3v3_LDO_Out"
+		(at 111.76 53.34 180)
 		(effects
 			(font
@@
 					(unit 1)
 				)
+			)
+		)
+	)
+	(symbol
+		(lib_id "power:PWR_FLAG")
+		(at 113.03 53.34 0)
+		(unit 1)
+		(body_style 1)
+		(exclude_from_sim no)
+		(in_bom yes)
+		(on_board yes)
+		(in_pos_files yes)
+		(dnp no)
+		(fields_autoplaced yes)
+		(property "Reference" "#FLG01003"
+			(at 113.03 51.435 0)
+			(hide yes)
+			(show_name no)
+			(do_not_autoplace no)
+			(effects
+				(font
+					(size 1.27 1.27)
+				)
+			)
+		)
+		(property "Value" "PWR_FLAG"
+			(at 113.03 48.26 0)
+			(show_name no)
+			(do_not_autoplace no)
+			(effects
+				(font
+					(size 1.27 1.27)
+				)
+			)
+		)
+		(property "Footprint" ""
+			(at 113.03 53.34 0)
+			(hide yes)
+			(show_name no)
+			(do_not_autoplace no)
+			(effects
+				(font
+					(size 1.27 1.27)
+				)
+			)
+		)
+		(property "Datasheet" ""
+			(at 113.03 53.34 0)
+			(hide yes)
+			(show_name no)
+			(do_not_autoplace no)
+			(effects
+				(font
+					(size 1.27 1.27)
+				)
+			)
+		)
+		(property "Description" "Special symbol for telling ERC where power comes from"
+			(at 113.03 53.34 0)
+			(hide yes)
+			(show_name no)
+			(do_not_autoplace no)
+			(effects
+				(font
+					(size 1.27 1.27)
+				)
+			)
+		)
+		(pin "1"
+		)
+		(instances
+			(project "mradio"
+				(path "/2cc0edad-946a-464e-a48b-49648a6334ed/e2cd56ff-e1ff-487d-8f44-743edfee6194"
+					(reference "#FLG01003")
+					(unit 1)
+				)

Commit message: LDO footprint updates
Parts:
- C1001, C1002, C1003, C1004: footprint RGR0020A -> Capacitor_SMD:C_0603_1608Metric
- C1005, C1006, C1007, C1008, C1009, C1010: footprint (none) -> Capacitor_SMD:C_0603_1608Metric
- D1001: footprint (none) -> LED_SMD:LED_0603_1608Metric
- R1001: footprint (none) -> Resistor_SMD:R_0603_1608Metric
- U1001: footprint RGR0020A -> TPS7A8500RGRR:RGR0020A
Connections:
- net 1V8_LDO_Out renamed +1V8
- net 2V_Buck_or_3v3_LDO_Out renamed +2V2
- net 3v3_LDO_Out renamed +3V3

Commit message: Update some footprints
Parts:
- TP1001: footprint Module:RaspberryPi_Pico_SMD -> TestPoint:TestPoint_Loop_D2.60mm_Drill0.9mm_Beaded
Changed lines of the file:
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@@
 			)
 		)
-		(property "Footprint" "Module:RaspberryPi_Pico_SMD"
+		(property "Footprint" "TestPoint:TestPoint_Loop_D2.60mm_Drill0.9mm_Beaded"
 			(at 157.48 83.82 0)
 			(hide yes)

Commit message: make test points smaller
Parts:
- TP1001: footprint TestPoint:TestPoint_Loop_D2.60mm_Drill0.9mm_Beaded -> TestPoint:TestPoint_Loop_D1.80mm_Drill1.0mm_Beaded
Changed lines of the file:
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@@
 			)
 		)
-		(property "Footprint" "TestPoint:TestPoint_Loop_D2.60mm_Drill0.9mm_Beaded"
+		(property "Footprint" "TestPoint:TestPoint_Loop_D1.80mm_Drill1.0mm_Beaded"
 			(at 157.48 83.82 0)
 			(hide yes)

Commit message: power conversion
Parts:
- renumbered C1001 to C901, C1002 to C902, C1003 to C903, C1004 to C904, C1005 to C905, C1006 to C906, C1007 to C907, C1008 to C908, C1009 to C909, C1010 to C910, D1001 to D901, R1001 to R901, TP1001 to TP901, U1001 to U901
Changed lines of the file:
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@@
 		(dnp no)
 		(fields_autoplaced yes)
-		(property "Reference" "C1001"
+		(property "Reference" "C901"
 			(at 71.12 76.1999 0)
 			(show_name no)
@@
 			(project "mradio"
 				(path "/2cc0edad-946a-464e-a48b-49648a6334ed/e2cd56ff-e1ff-487d-8f44-743edfee6194"
-					(reference "C1001")
+					(reference "C901")
 					(unit 1)
 				)
@@
 		(dnp no)
 		(fields_autoplaced yes)
-		(property "Reference" "C1002"
+		(property "Reference" "C902"
 			(at 82.55 76.1999 0)
 			(show_name no)
@@
 			(project "mradio"
 				(path "/2cc0edad-946a-464e-a48b-49648a6334ed/e2cd56ff-e1ff-487d-8f44-743edfee6194"
-					(reference "C1002")
+					(reference "C902")
 					(unit 1)
 				)
@@
 		(in_pos_files yes)
 		(dnp no)
-		(property "Reference" "#PWR01008"
+		(property "Reference" "#PWR0908"
 			(at 166.37 80.01 0)
 			(hide yes)
@@
 			(project "mradio"
 				(path "/2cc0edad-946a-464e-a48b-49648a6334ed/e2cd56ff-e1ff-487d-8f44-743edfee6194"
-					(reference "#PWR01008")
+					(reference "#PWR0908")
 					(unit 1)
 				)
@@
 		(dnp no)
 		(fields_autoplaced yes)
-		(property "Reference" "#PWR01006"
+		(property "Reference" "#PWR0906"
 			(at 115.57 53.34 0)
 			(hide yes)
@@
 			(project "mradio"
 				(path "/2cc0edad-946a-464e-a48b-49648a6334ed/e2cd56ff-e1ff-487d-8f44-743edfee6194"
-					(reference "#PWR01006")
+					(reference "#PWR0906")
 					(unit 1)
 				)
@@
 		(dnp no)
 		(fields_autoplaced yes)
-		(property "Reference" "#PWR01007"
+		(property "Reference" "#PWR0907"
 			(at 152.4 123.19 0)
 			(hide yes)
@@
 			(project "mradio"
 				(path "/2cc0edad-946a-464e-a48b-49648a6334ed/e2cd56ff-e1ff-487d-8f44-743edfee6194"
-					(reference "#PWR01007")
+					(reference "#PWR0907")
 					(unit 1)
 				)
@@
 		(dnp no)
 		(fields_autoplaced yes)
-		(property "Reference" "U1001"
+		(property "Reference" "U901"
 			(at 132.08 63.5 0)
 			(show_name no)
@@
 			(project "mradio"
 				(path "/2cc0edad-946a-464e-a48b-49648a6334ed/e2cd56ff-e1ff-487d-8f44-743edfee6194"
-					(reference "U1001")
+					(reference "U901")
 					(unit 1)
 				)
@@
 		(dnp no)
 		(fields_autoplaced yes)
-		(property "Reference" "#PWR01001"
+		(property "Reference" "#PWR0901"
 			(at 71.12 73.66 0)
 			(hide yes)
@@
 			(project "mradio"
 				(path "/2cc0edad-946a-464e-a48b-49648a6334ed/e2cd56ff-e1ff-487d-8f44-743edfee6194"
-					(reference "#PWR01001")
+					(reference "#PWR0901")
 					(unit 1)
 				)
@@
 		(dnp no)
 		(fields_autoplaced yes)
-		(property "Reference" "C1005"
+		(property "Reference" "C905"
 			(at 99.06 99.0599 0)
 			(show_name no)
@@
 			(project "mradio"
 				(path "/2cc0edad-946a-464e-a48b-49648a6334ed/e2cd56ff-e1ff-487d-8f44-743edfee6194"
-					(reference "C1005")
+					(reference "C905")
 					(unit 1)
 				)
@@
 		(dnp no)
 		(fields_autoplaced yes)
-		(property "Reference" "D1001"
+		(property "Reference" "D901"
 			(at 161.6075 66.04 0)
 			(show_name no)
@@
 			(project "mradio"
 				(path "/2cc0edad-946a-464e-a48b-49648a6334ed/e2cd56ff-e1ff-487d-8f44-743edfee6194"
-					(reference "D1001")
+					(reference "D901")
 					(unit 1)
 				)
@@
 		(dnp no)
 		(fields_autoplaced yes)
-		(property "Reference" "R1001"
+		(property "Reference" "R901"
 			(at 132.08 46.99 90)
 			(show_name no)
@@
 			(project "mradio"
 				(path "/2cc0edad-946a-464e-a48b-49648a6334ed/e2cd56ff-e1ff-487d-8f44-743edfee6194"
-					(reference "R1001")
+					(reference "R901")
 					(unit 1)
 				)
@@
 		(dnp no)
 		(fields_autoplaced yes)
-		(property "Reference" "C1006"
+		(property "Reference" "C906"
 			(at 171.45 96.5199 0)
 			(show_name no)
@@
 			(project "mradio"
 				(path "/2cc0edad-946a-464e-a48b-49648a6334ed/e2cd56ff-e1ff-487d-8f44-743edfee6194"
-					(reference "C1006")
+					(reference "C906")
 					(unit 1)
 				)
@@
 		(dnp no)
 		(fields_autoplaced yes)
-		(property "Reference" "#PWR01010"
+		(property "Reference" "#PWR0910"
 			(at 223.52 83.82 0)
 			(hide yes)
@@
 			(project "mradio"
 				(path "/2cc0edad-946a-464e-a48b-49648a6334ed/e2cd56ff-e1ff-487d-8f44-743edfee6194"
-					(reference "#PWR01010")
+					(reference "#PWR0910")
 					(unit 1)
 				)
@@
 		(dnp no)
 		(fields_autoplaced yes)
-		(property "Reference" "C1003"
+		(property "Reference" "C903"
 			(at 92.71 91.4399 0)
 			(show_name no)
@@
 			(project "mradio"
 				(path "/2cc0edad-946a-464e-a48b-49648a6334ed/e2cd56ff-e1ff-487d-8f44-743edfee6194"
-					(reference "C1003")
+					(reference "C903")
 					(unit 1)
 				)
@@
 		(dnp no)
 		(fields_autoplaced yes)
-		(property "Reference" "C1004"
+		(property "Reference" "C904"
 			(at 93.98 76.1999 0)
 			(show_name no)
@@
 			(project "mradio"
 				(path "/2cc0edad-946a-464e-a48b-49648a6334ed/e2cd56ff-e1ff-487d-8f44-743edfee6194"
-					(reference "C1004")
+					(reference "C904")
 					(unit 1)
 				)
@@
 		(dnp no)
 		(fields_autoplaced yes)
-		(property "Reference" "C1008"
+		(property "Reference" "C908"
 			(at 208.28 86.3599 0)
 			(show_name no)
@@
 			(project "mradio"
 				(path "/2cc0edad-946a-464e-a48b-49648a6334ed/e2cd56ff-e1ff-487d-8f44-743edfee6194"
-					(reference "C1008")
+					(reference "C908")
 					(unit 1)
 				)
@@
 		(dnp no)
 		(fields_autoplaced yes)
-		(property "Reference" "#PWR01009"
+		(property "Reference" "#PWR0909"
 			(at 191.77 100.33 0)
 			(hide yes)
@@
 			(project "mradio"
 				(path "/2cc0edad-946a-464e-a48b-49648a6334ed/e2cd56ff-e1ff-487d-8f44-743edfee6194"
-					(reference "#PWR01009")
+					(reference "#PWR0909")
 					(unit 1)
 				)
@@
 		(dnp no)
 		(fields_autoplaced yes)
-		(property "Reference" "#PWR01005"
+		(property "Reference" "#PWR0905"
 			(at 105.41 128.27 0)
 			(hide yes)
@@
 			(project "mradio"
 				(path "/2cc0edad-946a-464e-a48b-49648a6334ed/e2cd56ff-e1ff-487d-8f44-743edfee6194"
-					(reference "#PWR01005")
+					(reference "#PWR0905")
 					(unit 1)
 				)
@@
 		(dnp no)
 		(fields_autoplaced yes)
-		(property "Reference" "#PWR01003"
+		(property "Reference" "#PWR0903"
 			(at 88.9 102.87 0)
 			(hide yes)
@@
 			(project "mradio"
 				(path "/2cc0edad-946a-464e-a48b-49648a6334ed/e2cd56ff-e1ff-487d-8f44-743edfee6194"
-					(reference "#PWR01003")
+					(reference "#PWR0903")
 					(unit 1)
 				)
@@
 		(dnp no)
 		(fields_autoplaced yes)
-		(property "Reference" "C1007"
+		(property "Reference" "C907"
 			(at 195.58 86.3599 0)
 			(show_name no)
@@
 			(project "mradio"
 				(path "/2cc0edad-946a-464e-a48b-49648a6334ed/e2cd56ff-e1ff-487d-8f44-743edfee6194"
-					(reference "C1007")
+					(reference "C907")
 					(unit 1)
 				)
@@
 		(dnp no)
 		(fields_autoplaced yes)
-		(property "Reference" "TP1001"
+		(property "Reference" "TP901"
 			(at 154.94 79.2479 0)
 			(show_name no)
@@
 			(project "mradio"
 				(path "/2cc0edad-946a-464e-a48b-49648a6334ed/e2cd56ff-e1ff-487d-8f44-743edfee6194"
-					(reference "TP1001")
+					(reference "TP901")
 					(unit 1)
 				)
@@
 		(dnp no)
 		(fields_autoplaced yes)
-		(property "Reference" "C1010"
+		(property "Reference" "C910"
 			(at 231.14 86.3599 0)
 			(show_name no)
@@
 			(project "mradio"
 				(path "/2cc0edad-946a-464e-a48b-49648a6334ed/e2cd56ff-e1ff-487d-8f44-743edfee6194"
-					(reference "C1010")
+					(reference "C910")
 					(unit 1)
 				)
@@
 		(dnp no)
 		(fields_autoplaced yes)
-		(property "Reference" "#FLG01001"
+		(property "Reference" "#FLG0901"
 			(at 69.85 71.755 0)
 			(hide yes)
@@
 			(project "mradio"
 				(path "/2cc0edad-946a-464e-a48b-49648a6334ed/e2cd56ff-e1ff-487d-8f44-743edfee6194"
-					(reference "#FLG01001")
+					(reference "#FLG0901")
 					(unit 1)
 				)
@@
 		(dnp no)
 		(fields_autoplaced yes)
-		(property "Reference" "#PWR01002"
+		(property "Reference" "#PWR0902"
 			(at 67.31 91.44 0)
 			(hide yes)
@@
 			(project "mradio"
 				(path "/2cc0edad-946a-464e-a48b-49648a6334ed/e2cd56ff-e1ff-487d-8f44-743edfee6194"
-					(reference "#PWR01002")
+					(reference "#PWR0902")
 					(unit 1)
 				)
@@
 		(dnp no)
 		(fields_autoplaced yes)
-		(property "Reference" "C1009"
+		(property "Reference" "C909"
 			(at 219.71 86.3599 0)
 			(show_name no)
@@
 			(project "mradio"
 				(path "/2cc0edad-946a-464e-a48b-49648a6334ed/e2cd56ff-e1ff-487d-8f44-743edfee6194"
-					(reference "C1009")
+					(reference "C909")
 					(unit 1)
 				)
@@
 		(dnp no)
 		(fields_autoplaced yes)
-		(property "Reference" "#FLG01002"
+		(property "Reference" "#FLG0902"
 			(at 113.03 51.435 0)
 			(hide yes)
@@
 			(project "mradio"
 				(path "/2cc0edad-946a-464e-a48b-49648a6334ed/e2cd56ff-e1ff-487d-8f44-743edfee6194"
-					(reference "#FLG01002")
+					(reference "#FLG0902")
 					(unit 1)
 				)
@@
 		(dnp no)
 		(fields_autoplaced yes)
-		(property "Reference" "#PWR01004"
+		(property "Reference" "#PWR0904"
 			(at 95.25 110.49 0)
 			(hide yes)
@@
 			(project "mradio"
 				(path "/2cc0edad-946a-464e-a48b-49648a6334ed/e2cd56ff-e1ff-487d-8f44-743edfee6194"
-					(reference "#PWR01004")
-					(unit 1)
-				)
+					(reference "#PWR0904")
+					(unit 1)
+				)

Commit message: all traces routed
Parts:
- U901: footprint TPS7A8500RGRR:RGR0020A -> TPS7A8500RGRR:TPS7A8500RGRR
Changed lines of the file:
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@@
 			)
 		)
-		(property "Footprint" "TPS7A8500RGRR:RGR0020A"
+		(property "Footprint" "TPS7A8500RGRR:TPS7A8500RGRR"
 			(at 132.08 93.98 0)
 			(hide yes)
